File: keyfrick.kicad_pcb (KiCad board)
At the start: 2 copper layers, 96 x 34 mm, 13 parts, among them SW1 SW_Push, SW2 SW_Push, SW3 SW_Push, SW4 SW_Push, U1 XIAO-RP2040-DIP

Commit message: added fills lol
Routing:
- net GND: track 101.6 -> 0.06 mm
- added copper zone on F.Cu, net (none)
- added copper zone on B.Cu, net GND
Changed lines of the file:
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@@
 			(layer "F.SilkS")
 		)
-		(fp_circle
-			(center -3.2 0)
-			(end -3.1 0)
-			(stroke
-				(width 0.2)
-				(type solid)
-			)
-			(fill no)
-			(layer "F.SilkS")
-		)
 		(fp_line
 			(start -2.75 -1.64)
@@
 			(layer "F.SilkS")
 		)
-		(fp_circle
-			(center -3.2 0)
-			(end -3.1 0)
-			(stroke
-				(width 0.2)
-				(type solid)
-			)
-			(fill no)
-			(layer "F.SilkS")
-		)
 		(fp_line
 			(start -2.75 -1.64)
@@
 			(layer "F.SilkS")
 		)
-		(fp_circle
-			(center -3.2 0)
-			(end -3.1 0)
-			(stroke
-				(width 0.2)
-				(type solid)
-			)
-			(fill no)
-			(layer "F.SilkS")
-		)
 		(fp_line
 			(start -2.75 -1.64)
@@
 			(layer "F.SilkS")
 		)
-		(fp_circle
-			(center -8.95 -10.3)
-			(end -8.95 -10.554)
-			(stroke
-				(width 0.5)
-				(type solid)
-			)
-			(fill yes)
-			(layer "F.SilkS")
-		)
 		(fp_rect
 			(start -8.9 -10.55)
@@
 			(layer "F.SilkS")
 		)
-		(fp_circle
-			(center -3.2 0)
-			(end -3.1 0)
-			(stroke
-				(width 0.2)
-				(type solid)
-			)
-			(fill no)
-			(layer "F.SilkS")
-		)
 		(fp_line
 			(start -2.75 -1.64)
@@
 	)
 	(segment
-		(start 158.73 54.96)
-		(end 156.19 57.5)
-		(width 0.2)
-		(layer "B.Cu")
-		(net 1)
-	)
-	(segment
-		(start 103.23 47)
-		(end 103.23 54.92)
-		(width 0.2)
-		(layer "B.Cu")
-		(net 1)
-	)
-	(segment
-		(start 119.19 57.46)
-		(end 100.69 57.46)
-		(width 0.2)
-		(layer "B.Cu")
-		(net 1)
-	)
-	(segment
 		(start 156.15 57.46)
 		(end 156.19 57.5)
@@
 	)
 	(segment
-		(start 103.23 54.92)
-		(end 100.69 57.46)
-		(width 0.2)
-		(layer "B.Cu")
-		(net 1)
-	)
-	(segment
-		(start 121.73 54.92)
-		(end 119.19 57.46)
-		(width 0.2)
-		(layer "B.Cu")
-		(net 1)
-	)
-	(segment
-		(start 140.23 47)
-		(end 140.23 54.92)
-		(width 0.2)
-		(layer "B.Cu")
-		(net 1)
-	)
-	(segment
-		(start 140.23 54.92)
-		(end 137.69 57.46)
-		(width 0.2)
-		(layer "B.Cu")
-		(net 1)
-	)
-	(segment
-		(start 121.73 47)
-		(end 121.73 54.92)
-		(width 0.2)
-		(layer "B.Cu")
-		(net 1)
-	)
-	(segment
-		(start 158.73 47)
-		(end 158.73 54.96)
-		(width 0.2)
-		(layer "B.Cu")
-		(net 1)
-	)
-	(segment
-		(start 137.69 57.46)
-		(end 156.15 57.46)
-		(width 0.2)
-		(layer "B.Cu")
-		(net 1)
-	)
-	(segment
-		(start 119.19 57.46)
-		(end 137.69 57.46)
-		(width 0.2)
-		(layer "B.Cu")
-		(net 1)
-	)
-	(segment
 		(start 105.77 47)
 		(end 111.46 47)
@@
 		(net 13)
 	)
+	(zone
+		(net 0)
+		(net_name "")
+		(layer "F.Cu")
+		(hatch edge 0.5)
+		(priority 1)
+		(connect_pads
+			(clearance 0.5)
+		)
+		(min_thickness 0.25)
+		(filled_areas_thickness no)
+		(fill yes
+			(thermal_gap 0.5)
+			(thermal_bridge_width 0.5)
+			(island_removal_mode 1)
+			(island_area_min 10)
+		)
+		(polygon
+			(pts
+				(xy 95 43) (xy 95 77) (xy 191 77) (xy 191 43)
+			)
+		)
+	)
+	(zone
+		(net 1)
+		(net_name "GND")
+		(layer "B.Cu")
+		(hatch edge 0.5)
+		(connect_pads
+			(clearance 0.5)
+		)
+		(min_thickness 0.25)
+		(filled_areas_thickness no)
+		(fill yes
+			(thermal_gap 0.5)
+			(thermal_bridge_width 0.5)
+		)
+		(polygon
+			(pts
+				(xy 95 43) (xy 95 77) (xy 191 77) (xy 191 43)
+			)
+		)
+	)
 	(embedded_fonts no)

Commit message: Add files via upload
Parts:
- turned U1 to 0 degrees
Routing:
- net d1: track 89.6 -> 78.3 mm
- net sw3: track 33.1 -> 43.0 mm
- net sw2: track 55.4 -> 64.8 mm
- net sw1: track 77.6 -> 86.8 mm
- net d2: track 71.1 -> 62.6 mm
- net sw4: track 10.9 -> 17.2 mm
- net d3: track 50.4 -> 46.0 mm
- net d4: track 32.3 -> 28.4 mm

Commit message: completed project upload
Other:
- board text added: "+[----->+++<]>+++ +.------.[--->+<] >++.--[->+++<]>+. ---[->+++<]>+.-[- -->+<]>.++++++++."
- board text added: "keyf*ck"
